File: wch32v305pad.kicad_pcb (KiCad board)
At the start: 2 copper layers, 38.1 x 38.1 mm, 22 parts, among them J1 USB_C_Receptacle_USB2.0, J2 SWD, J3 UART, J4 Debug, SW1 SW_Push, SW10 Reset, SW2 SW_Push, SW3 SW_Push, SW4 SW_Push, U1 CH32V30xFxPx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

Commit message: Routing cleanups, some ignored files.
Parts:
- moved C2 0.32 mm to (58.7, 43.5)
Routing:
- net GND: track 39.1 -> 41.6 mm, vias 9 -> 10
