File: wch32v305pad.kicad_sch (KiCad schematic)
At the start: 22 parts, among them J1 USB_C_Receptacle_USB2.0, J2 SWD, J3 UART, J4 Debug, SW1 SW_Push, SW10 Reset, SW2 SW_Push, SW3 SW_Push, SW4 SW_Push, U1 CH32V30xFxPx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

Commit message: BOM fixes.
Parts:
- C3, C4: LCSC Part Number (none) -> C5186910
- J3, J4: LCSC Part Number (none) -> C160403
- R1, R2: LCSC Part Number (none) -> C27834
- SW1, SW2, SW3, SW4: now left out of the parts list
- U1: LCSC Part Number (none) -> C5123443
Changed lines of the file:
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@@
+			)
+		)
+		(property "LCSC Part Number" "C5186910"
+			(at 247.65 127 90)
+			(effects
+				(font
+					(size 1.27 1.27)
+				)
+				(hide yes)
 			)
 		)
@@
 		(unit 1)
 		(exclude_from_sim no)
-		(in_bom yes)
+		(in_bom no)
 		(on_board yes)
 		(dnp no)
@@
 		(unit 1)
 		(exclude_from_sim no)
-		(in_bom yes)
+		(in_bom no)
 		(on_board yes)
 		(dnp no)
@@
 			)
 		)
+		(property "LCSC Part Number" "C5123443"
+			(at 245.11 81.28 0)
+			(effects
+				(font
+					(size 1.27 1.27)
+				)
+				(hide yes)
+			)
+		)
 		(pin "16"
 		)
@@
 			)
 		)
+		(property "LCSC Part Number" "C5186910"
+			(at 247.65 121.92 90)
+			(effects
+				(font
+					(size 1.27 1.27)
+				)
+				(hide yes)
+			)
+		)
 		(pin "2"
 		)
@@
 			)
 		)
-		(property "LCSC Part Number" ""
+		(property "LCSC Part Number" "C27834"
 			(at 80.01 82.55 0)
 			(effects
@@
 			)
 		)
-		(property "LCSC Part Number" ""
+		(property "LCSC Part Number" "C27834"
 			(at 80.01 80.01 0)
 			(effects
@@
 		(unit 1)
 		(exclude_from_sim no)
-		(in_bom yes)
+		(in_bom no)
 		(on_board yes)
 		(dnp no)
@@
 			)
 		)
+		(property "LCSC Part Number" "C160403"
+			(at 215.9 25.4 0)
+			(effects
+				(font
+					(size 1.27 1.27)
+				)
+				(hide yes)
+			)
+		)
 		(pin "1"
 		)
@@
 		(unit 1)
 		(exclude_from_sim no)
-		(in_bom yes)
+		(in_bom no)
 		(on_board yes)
 		(dnp no)
@@
 			(at 217.17 39.37 0)
 			(effects
+				(font
+					(size 1.27 1.27)
+				)
+				(hide yes)
+			)
+		)
+		(property "LCSC Part Number" "C160403"
+			(at 217.17 39.37 0)
+			(effects

Commit message: Routing cleanups, some ignored files.
Parts:
- C3, C4: LCSC Part Number C5186910 -> C1816
- J1: LCSC Part Number C3001293 -> C2843967
- SW10: LCSC Part Number C388858 -> C79175; MPN SKQGAKE020 -> EVQPUC02K
Changed lines of the file:
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@@
 			)
 		)
-		(property "LCSC Part Number" "C5186910"
+		(property "LCSC Part Number" "C1816"
 			(at 247.65 127 90)
 			(effects
@@
 			)
 		)
-		(property "LCSC Part Number" "C3001293"
+		(property "LCSC Part Number" "C2843967"
 			(at 49.53 90.17 0)
 			(effects
@@
 			)
 		)
-		(property "LCSC Part Number" "C5186910"
+		(property "LCSC Part Number" "C1816"
 			(at 247.65 121.92 90)
 			(effects
@@
 			)
 		)
-		(property "LCSC Part Number" "C388858"
+		(property "LCSC Part Number" "C79175"
 			(at 149.86 152.4 0)
 			(effects
@@
 			)
 		)
-		(property "MPN" "SKQGAKE020"
+		(property "MPN" "EVQPUC02K"
 			(at 149.86 152.4 0)
 			(effects
